Commit message: chroe(parameters): Renamed thhe name of a file and changing in the parameters

File: robot_gazebo/model/robot_drone_gazebo.urdf.xacro (robot description, xacro)
@@ -2,7 +2,7 @@
 <robot xmlns:xacro="http://www.ros.org/wiki/xacro" name="X3">
     <xacro:arg name="simulation_config_file" default="$(find robot_gazebo)/config/simulation_config.yaml" />
-    <xacro:arg name="simulation_config_file" default="$(find robot_gazebo)/config/sensors_and_perception_config.yaml" />
-    <xacro:include filename="$(find robot_gazebo)/model/sensors_and_perception_macros.xacro"/>
+    <xacro:arg name="simulation_config_file" default="$(find robot_gazebo)/config/geometry_sensing_config.yaml" />
+    <xacro:include filename="$(find robot_gazebo)/model/robot_sensing_macros.xacro"/>
     <xacro:property name="sim_config_file" value="$(arg simulation_config_file)"/>
-    <xacro:property name="sim_config_file" value="$(xacro.load_yaml(sim_config_file))"//>
+    <xacro:property name="sim_config_values" value="$(xacro.load_yaml(sim_config_file))"//>
 </robot>

File: robot_gazebo/model/robot_drone_geometry.urdf.xacro (robot description, xacro)
@@ -1,10 +1,10 @@
 <?xml version="1.0"?>
 <robot xmlns:xacro="http://www.ros.org/wiki/xacro" name="X3">
-    <xacro:arg name="geometry_config_file" default="$(find robot_gazebo)/config/geometry_drone_config.yaml"/>
-    <xacro:arg name="geometry_config_file" default="$(find robot_gazebo)/config/geometry_sensing_config.yaml"/>
+    <xacro:arg name="geometry_robot_config_file" default="$(find robot_gazebo)/config/geometry_drone_config.yaml"/>
+    <xacro:arg name="geometry_sensing_config_file" default="$(find robot_gazebo)/config/geometry_sensing_config.yaml"/>
     <xacro:include filename="$(find robot_gazebo)/model/brushless_rotor.urdf.xacro">
     <xacro:include filename="$(find robot_gazebo)/model/inertial_macros.xacro">
-    <xacro:include filename="$(find robot_gazebo)/model/sensing_and_perception_macros.xacro">
-    <xacro:property name="config_file" value="$(arg geometry_config_file)">
+    <xacro:include filename="$(find robot_gazebo)/model/robot_sensing_macros.xacro">
+    <xacro:property name="config_file" value="$(arg geometry_robot_config_file)">
     <link name="base_link"/>
     <xacro:brushless_rotor>
@@ -12,35 +12,51 @@
         parent="base_link"
         child="rotor_0"
-        lower_limit:=-1e+16
-        upper_limit:=1e+16
-        rotor_drive_radius:=0.1
-        rotor_drive_length:=0.005
+        lower_limit:=lower_limit
+        upper_limit:=upper_limit
+        rotor_drive_radius:=rotor_drive_radius
+        rotor_drive_length:=rotor_drive_length
         drive_color:=red
+        roto_mass:=rotor_mass
+        roto_x:= position_x
+        roto_y:= -position_y
+        roto_z:= position_z
     <xacro:brushless_rotor>
         name="rotor_1"
         parent="base_link"
         child="rotor_1"
-        lower_limit:=-1e+16
-        upper_limit:=1e+16
-        rotor_drive_radius:=0.1
-        rotor_drive_length:=0.005
+        lower_limit:=lower_limit
+        upper_limit:=upper_limit
+        rotor_drive_radius:=rotor_drive_radius
+        rotor_drive_length:=rotor_drive_length
         drive_color:=red
+        roto_mass:=rotor_mass
+        roto_x:= -position_x
+        roto_y:= position_y
+        roto_z:= position_z
     <xacro:brushless_rotor>
         name="rotor_2"
         parent="base_link"
         child="rotor_2"
-        lower_limit:=-1e+16
-        upper_limit:=1e+16
-        rotor_drive_radius:=0.1
-        rotor_drive_length:=0.005
+        lower_limit:=lower_limit
+        upper_limit:=upper_limit
+        rotor_drive_radius:=rotor_drive_radius
+        rotor_drive_length:=rotor_drive_length
         drive_color:=red
+        roto_mass:=rotor_mass
+        roto_x:= position_x
+        roto_y:= position_y
+        roto_z:= position_z
     <xacro:brushless_rotor>
         name="rotor_3"
         parent="base_link"
         child="rotor_3"
-        lower_limit:=-1e+16
-        upper_limit:=1e+16
-        rotor_drive_radius:=0.1
-        rotor_drive_length:=0.005
+        lower_limit:=lower_limit
+        upper_limit:=upper_limit
+        rotor_drive_radius:=rotor_drive_radius
+        rotor_drive_length:=rotor_drive_length
         drive_color:=red
+        roto_mass:=rotor_mass
+        roto_x:= -position_x
+        roto_y:= -position_y
+        roto_z:= position_z
 </robot>
